Commit message: added gazebo

File: upcreate3_description/urdf/parts/realsense_bracket.urdf.xacro (robot description, xacro)
@@ -1,38 +1,40 @@
 <?xml version="1.0"?>
-<robot name="realsense_bracket" xmlns:xacro="http://ros.org/wiki/xacro">
-    <xacro:property name="M_PI" value="3.1415926535897931" />
-    <xacro:property name="M_PI_2" value="1.570796327" />
-    <gazebo reference="realsense_bracket_base">
-        <material>Gazebo/Blue</material>
-    </gazebo>
-    <material name="light_blue">
-        <color rgba="0 0.5 1.0 1"/>
-    </material>
-    <link name="realsense_bracket_base">
-        <visual>
-            <origin xyz="0.078 0 -0.054" rpy="${M_PI_2} 0 ${M_PI_2}"/>
-            <geometry>
-                <mesh filename="package://upcreate3_description/meshes/C3-RealSense-D435-Mount.stl" scale="0.001 0.001 0.001"/>
-            </geometry>
-            <material name="light_blue"/>
-        </visual>
-        <collision>
-            <origin xyz="0 0 0" rpy="0 0 0" />
-            <geometry>
-                <box size="0.1 0.1 0.1"/>
-            </geometry>
-        </collision>
-        <inertial>
-            <mass value="0.001" />
-            <origin xyz="0 0 0" />
-            <inertia ixx="0.001" ixy="0.0" ixz="0.0" iyy="0.001" iyz="0.0" izz="0.001" />
-      </inertial>
-    </link>
-    <link name="realsense_bracket_camera_mount">
-    </link>
-    <joint name="realsense_bracket_joint" type="fixed">
-      <origin xyz="0.047 0.0 0.0895" rpy="0 0 0"/>
-      <parent link="realsense_bracket_base"/>
-      <child link="realsense_bracket_camera_mount" />
-    </joint>
+<robot xmlns:xacro="http://ros.org/wiki/xacro">
+    <xacro:macro name="realsense_bracket">
+        <xacro:property name="M_PI" value="3.1415926535897931" />
+        <xacro:property name="M_PI_2" value="1.570796327" />
+        <gazebo reference="realsense_bracket_base">
+            <material>Gazebo/Blue</material>
+        </gazebo>
+        <material name="light_blue">
+            <color rgba="0 0.5 1.0 1"/>
+        </material>
+        <link name="realsense_bracket_base">
+            <visual>
+                <origin xyz="0.078 0 -0.054" rpy="${M_PI_2} 0 ${M_PI_2}"/>
+                <geometry>
+                    <mesh filename="package://upcreate3_description/meshes/C3-RealSense-D435-Mount.stl" scale="0.001 0.001 0.001"/>
+                </geometry>
+                <material name="light_blue"/>
+            </visual>
+            <collision>
+                <origin xyz="0 0 0" rpy="0 0 0" />
+                <geometry>
+                    <box size="0.1 0.1 0.1"/>
+                </geometry>
+            </collision>
+            <inertial>
+                <mass value="0.001" />
+                <origin xyz="0 0 0" />
+                <inertia ixx="0.001" ixy="0.0" ixz="0.0" iyy="0.001" iyz="0.0" izz="0.001" />
+        </inertial>
+        </link>
+        <link name="realsense_bracket_camera_mount">
+        </link>
+        <joint name="realsense_bracket_joint" type="fixed">
+            <origin xyz="0.047 0.0 0.0895" rpy="0 0 0"/>
+            <parent link="realsense_bracket_base"/>
+            <child link="realsense_bracket_camera_mount" />
+        </joint>
+    </xacro:macro>
 </robot>

File: upcreate3_description/urdf/sensors/realsense.urdf.xacro (robot description, xacro)
@@ -7,3 +7,56 @@
     <origin xyz="0 0 0" rpy="0 0 0"/>
   </xacro:sensor_d435>
+  <gazebo reference="camera_link">
+    <material>Gazebo/Grey</material>
+  </gazebo>
+  <gazebo reference="camera_link">
+    <sensor name="d435" type="depth">
+        <update_rate>30</update_rate>
+        <camera>
+            <horizontal_fov>1.59174</horizontal_fov>
+            <image>
+                <width>640</width>
+                <height>480</height>
+                <format>R8G8B8</format>
+            </image>
+            <clip>
+              <near>0.02</near>
+              <far>6.0</far>
+            </clip>
+            <distortion>
+              <k1>0</k1>
+              <k2>0</k2>
+              <k3>0</k3>
+              <k4>0</k4>
+              <k5>0</k5>
+              <center>0 0</center>
+            </distortion>
+        </camera>
+        <plugin name="camera_plugin" filename="libgazebo_ros_camera.so">
+            <visualize>true</visualize>
+            <baseline>0.05</baseline>
+            <alwaysOn>true</alwaysOn>
+            <updateRate>0.0</updateRate>
+            <cameraName>camera</cameraName>
+            <ros>
+              <namespace>camera</namespace>
+              <remapping>custom_camera/image_raw:=camera/color/image_raw</remapping>
+              <remapping>custom_camera/image_depth:=camera/aligned_depth_to_color/image_raw</remapping>
+              <remapping>custom_camera/camera_info:=camera/color/camera_info</remapping>
+              <remapping>custom_camera/camera_info_depth:=camera/depth/camera_info</remapping>
+              <remapping>custom_camera/points:=camera/depth/color/points</remapping>
+            </ros>
+            <frameName>camera_link</frameName>
+            <pointCloudCutoff>0.2</pointCloudCutoff>
+            <pointCloudCutoffMax>6.0</pointCloudCutoffMax>
+            <focalLength>0</focalLength>
+            <hackBaseline>0</hackBaseline>
+            <CxPrime>0</CxPrime>
+            <Cx>0</Cx>
+            <Cy>0</Cy>
+            <min_depth>0.02</min_depth>
+            <max_depth>6.0</max_depth>
+        </plugin>
+    </sensor>
+  </gazebo>
 </robot>

File: upcreate3_description/urdf/upcreate3.urdf.xacro (robot description, xacro)
@@ -9,10 +9,11 @@
   <!-- Bracket for Realsense camera -->
   <xacro:include filename="$(find upcreate3_description)/urdf/parts/realsense_bracket.urdf.xacro" />
-  <joint name="realsense_bracket_base_joint" type="fixed">
-      <origin xyz="${BRACKET_GRID_X*CREATE3_GRID}  ${BRACKET_GRID_Y*CREATE3_GRID} ${CREATE3_TOP_Z}" rpy="0 0 0"/>
-      <parent link="base_link"/>
-      <child link="realsense_bracket_base" />
-  </joint>
   <!-- Realsense -->
   <xacro:include filename="$(find upcreate3_description)/urdf/sensors/realsense.urdf.xacro" />
+  <xacro:realsense_bracket />
+    <joint name="realsense_bracket_base_joint" type="fixed">
+        <origin xyz="${BRACKET_GRID_X*CREATE3_GRID}  ${BRACKET_GRID_Y*CREATE3_GRID} ${CREATE3_TOP_Z}" rpy="0 0 0"/>
+        <parent link="base_link"/>
+        <child link="realsense_bracket_base" />
+    </joint>
 </robot>
