Commit message: fixed realsense topics in gazebo

File: upcreate3_description/urdf/sensors/realsense.urdf.xacro (robot description, xacro)
@@ -4,4 +4,5 @@
   <xacro:arg name="use_mesh" default="true" />
   <xacro:include filename="$(find upcreate3_description)/urdf/sensors/realsense/d435.urdf.xacro" />
+  <xacro:property name="camera_name"  value="d435"/>
   <xacro:sensor_d435 parent="realsense_bracket_camera_mount" use_nominal_extrinsics="$(arg use_nominal_extrinsics)" use_mesh="$(arg use_mesh)">
     <origin xyz="0 0 0" rpy="0 0 0"/>
@@ -11,5 +12,5 @@
   </gazebo>
   <gazebo reference="camera_link">
-    <sensor name="d435" type="depth">
+    <sensor name="${camera_name}" type="depth">
         <update_rate>30</update_rate>
         <camera>
@@ -40,10 +41,10 @@
             <cameraName>camera</cameraName>
             <ros>
-              <namespace>camera</namespace>
-              <remapping>custom_camera/image_raw:=camera/color/image_raw</remapping>
-              <remapping>custom_camera/image_depth:=camera/aligned_depth_to_color/image_raw</remapping>
-              <remapping>custom_camera/camera_info:=camera/color/camera_info</remapping>
-              <remapping>custom_camera/camera_info_depth:=camera/depth/camera_info</remapping>
-              <remapping>custom_camera/points:=camera/depth/color/points</remapping>
+              <!--<namespace>camera</namespace>-->
+              <remapping>${camera_name}/image_raw:=camera/color/image_raw</remapping>
+              <remapping>${camera_name}/camera_info:=camera/color/camera_info</remapping>
+              <remapping>${camera_name}/depth/image_raw:=camera/aligned_depth_to_color/image_raw</remapping>
+              <remapping>${camera_name}/depth/camera_info:=camera/depth/camera_info</remapping>
+              <remapping>${camera_name}/points:=camera/depth/color/points</remapping>
             </ros>
             <frameName>camera_link</frameName>
